Commit message: Declared the FLS in the sensors urdf description
Declared the fls in eca_a9/eca_a9_description/urdf/eca_a9_sensors.xacro by inputting necessary parameters specified in uuv_simulator/uuv_sensor_plugins/uuv_sensor_ros_plugins/urdf/sonar_snippets.xacro

PROBLEM: TFs are OK but fls does not seem to be functional, i.e. no fls live feed in gazebo/rviz.

File: eca_a9/eca_a9_description/urdf/eca_a9_sensors.xacro (robot description, xacro)
@@ -37,4 +37,19 @@
       power_load="25"
       topic="${namespace}/dvl/state"/>
+    <!-- Forward Looking Sonar -->
+    <xacro:forward_looking_sonar
+      namespace="${namespace}"
+      suffix=""
+      parent_link="${namespace}/base_link"
+      topic="forward_sonar"
+      mass="0.015"
+      update_rate="10"
+      samples="100"
+      fov="1.54719755"
+      width="260"
+      height="120">
+      <inertia ixx="0.00001" ixy="0.0" ixz="0.0" iyy="0.00001" iyz="0.0" izz="0.00001" />
+      <origin xyz="0.83 0 -0.22" rpy="0 ${0.2*pi} 0" />
+    </xacro:forward_looking_sonar>
     <!-- Side scan sonar left -->
     <xacro:sidescan_sonar namespace="${namespace}" parent_link="${namespace}/base_link" suffix="left">
